File: kicad/proto_breadboard2/proto_breadboard2.kicad_sch (KiCad schematic)
At the start: 20 parts, among them J1 ISP header, SW1 SW_DPDT_x2, SW2 SW_MEC_5G, SW3 SW_MEC_5G, SW4 SW_MEC_5G, SW5 SW_MEC_5G, U2 ATtiny10, U3 12V boost converter

Commit message: playable brik.S; resistor ladder change for wider voltage gap between keys
Parts:
- removed R8: 2K2, symbol Device:R
- R3: value 8K2 -> 12K
- R4: value 4K7 -> 510K
- R5: value 2K2 -> 4K7
- R6: value 2K2 -> 8K2
- R7: value 8K2 -> 32K
Connections:
- net at R5.2, SW2.3 (B), SW2.4 (B): now also JP2.1 (A), R3.2, R4.1
Changed lines of the file:
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@@
-	(wire
-		(pts
-			(xy 111.76 138.43) (xy 111.76 140.335)
-		)
-		(stroke
-			(width 0)
-			(type default)
-		)
-	)
 	(wire
 		(pts
@@
 	(wire
 		(pts
-			(xy 111.76 147.955) (xy 111.76 149.86)
+			(xy 111.76 138.43) (xy 111.76 149.86)
 		)
 		(stroke
@@
 			)
 		)
-		(property "Value" "2K2"
+		(property "Value" "4K7"
 			(at 113.665 156.845 0)
 			(effects
@@
 			)
 		)
-		(property "Value" "4K7"
+		(property "Value" "510K"
 			(at 118.11 135.255 90)
 			(effects
@@
 			)
 		)
-		(property "Value" "8K2"
+		(property "Value" "12K"
 			(at 105.41 135.255 90)
 			(effects
@@
 	(symbol
 		(lib_id "Device:R")
-		(at 111.76 144.145 180)
-		(unit 1)
-		(exclude_from_sim no)
-		(in_bom yes)
-		(on_board yes)
-		(dnp no)
-		(fields_autoplaced yes)
-		(property "Reference" "R8"
-			(at 113.665 142.875 0)
-			(effects
-				(font
-					(size 1.27 1.27)
-				)
-				(justify right)
-			)
-		)
-		(property "Value" "2K2"
-			(at 113.665 145.415 0)
-			(effects
-				(font
-					(size 1.27 1.27)
-				)
-				(justify right)
-			)
-		)
-		(property "Footprint" ""
-			(at 113.538 144.145 90)
-			(effects
-				(font
-					(size 1.27 1.27)
-				)
-				(hide yes)
-			)
-		)
-		(property "Datasheet" "~"
-			(at 111.76 144.145 0)
-			(effects
-				(font
-					(size 1.27 1.27)
-				)
-				(hide yes)
-			)
-		)
-		(property "Description" ""
-			(at 111.76 144.145 0)
-			(effects
-				(font
-					(size 1.27 1.27)
-				)
-			)
-		)
-		(pin "2"
-		)
-		(pin "1"
-		)
-		(instances
-			(project "proto_breadboard"
-				(path "/9121eaa1-199f-4b0a-955e-7211dee87885"
-					(reference "R8")
-					(unit 1)
-				)
-			)
-		)
-	)
-	(symbol
-		(lib_id "Device:R")
 		(at 111.76 167.005 180)
 		(unit 1)
@@
 			)
 		)
-		(property "Value" "2K2"
+		(property "Value" "8K2"
 			(at 113.665 168.275 0)
 			(effects
@@
 			)
 		)
-		(property "Value" "8K2"
+		(property "Value" "32K"
 			(at 113.665 179.705 0)
 			(effects
