File: kicad/base_board2/base_board2.kicad_pcb (KiCad board)
At the start: 4 copper layers, 36.7 x 24.1 mm, 26 parts, among them J1 Conn_02x04_Odd_Even, J2 Conn_01x02, SW1 SW_Push, SW2 SW_Push, SW3 SW_Push, SW4 SW_Push, U1 IS31FL3743A, U2 LED matrix 15x10

Commit message: fix an oopsie on base_board2
Parts:
- removed the R6 at (140.4, 69.8)
- R4: value 8K2 -> 15K
- R6: renamed from R7; value 2K2 -> 4K7
- R7: renamed from R8; value 2K2 -> 10K
- R8: renamed from R9; value 8K2 -> 47K
- R9: renamed from R10; value 4K7 -> 680K
- moved R9 1.60 mm to (140.4, 68.2)
- moved R4 1.60 mm to (140.4, 69.8)
- renumbered R11 to R10
Connections:
- R6 pad 1: Net-(R6-Pad2) (its old number) -> ATTINY_PB0
- SW1 pad 2: Net-(R6-Pad2) (its old number) -> ATTINY_PB0
- U1 pad 26: SDB -> VCC
Routing:
- net Net-(R6-Pad2) (its old number): track 40.0 -> 0.00 mm, vias 2 -> 0
- net ATTINY_PB0: track 27.8 -> 67.0 mm, vias 2 -> 4
- net VCC: track 68.0 -> 72.6 mm
- net GND: track 43.7 -> 44.9 mm
