File: kicad/power_supply/power_supply.kicad_sch (KiCad schematic)
At the start: 18 parts, among them J1 USB_C_Receptacle_PowerOnly_6P, J2 Battery terminal, J3 Base board terminal, Q1 DMG2301L, U1 MCP1640x-xCHY, U2 MCP73831-2-OT

Commit message: pcbs: improve powering scheme, redesign cartridge; 3dcad: update whole housing
Parts:
- added J4: Shorted if cartridge present, components:Pads_1x2mm_2x, symbol Connector_Generic:Conn_01x02
- J3: value Base board terminal -> Base board power terminal
Connections:
- net VSYS: now also J4.2 (Pin_2); no longer U1.3 (EN)
- new net: J4.1 (Pin_1), U1.3 (EN)
Changed lines of the file:
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@@
+		(color 0 0 0 0)
+	)
+	(junction
+		(at 105.41 128.27)
+		(diameter 0)
 		(color 0 0 0 0)
 	)
@@
 	(wire
 		(pts
-			(xy 129.54 133.35) (xy 121.92 133.35)
-		)
-		(stroke
-			(width 0)
-			(type default)
-		)
-	)
-	(wire
-		(pts
 			(xy 139.7 140.97) (xy 139.7 151.13)
 		)
@@
 	(wire
 		(pts
+			(xy 121.92 133.35) (xy 129.54 133.35)
+		)
+		(stroke
+			(width 0)
+			(type default)
+		)
+	)
+	(wire
+		(pts
 			(xy 80.01 58.42) (xy 71.12 58.42)
 		)
@@
 	(wire
 		(pts
-			(xy 97.79 128.27) (xy 111.76 128.27)
+			(xy 97.79 146.05) (xy 121.92 146.05)
+		)
+		(stroke
+			(width 0)
+			(type default)
+		)
+	)
+	(wire
+		(pts
+			(xy 97.79 128.27) (xy 105.41 128.27)
 		)
 		(stroke
@@
 	(wire
 		(pts
+			(xy 105.41 143.51) (xy 105.41 128.27)
+		)
+		(stroke
+			(width 0)
+			(type default)
+		)
+	)
+	(wire
+		(pts
+			(xy 105.41 128.27) (xy 111.76 128.27)
+		)
+		(stroke
+			(width 0)
+			(type default)
+		)
+	)
+	(wire
+		(pts
 			(xy 41.91 80.01) (xy 41.91 87.63)
 		)
@@
 	(wire
 		(pts
+			(xy 97.79 143.51) (xy 105.41 143.51)
+		)
+		(stroke
+			(width 0)
+			(type default)
+		)
+	)
+	(wire
+		(pts
 			(xy 111.76 138.43) (xy 111.76 151.13)
 		)
@@
 	(wire
 		(pts
-			(xy 121.92 133.35) (xy 121.92 128.27)
-		)
-		(stroke
-			(width 0)
-			(type default)
-		)
-	)
-	(wire
-		(pts
 			(xy 246.38 76.2) (xy 234.95 76.2)
 		)
@@
 		(pts
 			(xy 41.91 87.63) (xy 34.29 87.63)
+		)
+		(stroke
+			(width 0)
+			(type default)
+		)
+	)
+	(wire
+		(pts
+			(xy 121.92 146.05) (xy 121.92 133.35)
 		)
 		(stroke
@@
 			)
 		)
-		(property "Value" "Base board terminal"
+		(property "Value" "Base board power terminal"
 			(at 204.47 124.4599 0)
 			(effects
@@
 					(unit 1)
 				)
+			)
+		)
+	)
+	(symbol
+		(lib_id "Connector_Generic:Conn_01x02")
+		(at 92.71 146.05 180)
+		(unit 1)
+		(exclude_from_sim no)
+		(in_bom yes)
+		(on_board yes)
+		(dnp no)
+		(property "Reference" "J4"
+			(at 92.71 137.16 0)
+			(effects
+				(font
+					(size 1.27 1.27)
+				)
+			)
+		)
+		(property "Value" "Shorted if cartridge present"
+			(at 89.916 139.954 0)
+			(effects
+				(font
+					(size 1.27 1.27)
+				)
+			)
+		)
+		(property "Footprint" "components:Pads_1x2mm_2x"
+			(at 92.71 146.05 0)
+			(effects
+				(font
+					(size 1.27 1.27)
+				)
+				(hide yes)
+			)
+		)
+		(property "Datasheet" "~"
+			(at 92.71 146.05 0)
+			(effects
+				(font
+					(size 1.27 1.27)
+				)
+				(hide yes)
+			)
+		)
+		(property "Description" "Generic connector, single row, 01x02, script generated (kicad-library-utils/schlib/autogen/connector/)"
+			(at 92.71 146.05 0)
+			(effects
+				(font
+					(size 1.27 1.27)
+				)
+				(hide yes)
+			)
+		)
+		(pin "2"
+		)
+		(pin "1"
+		)
+		(instances
+			(project "power_supply"
+				(path "/5e0ffdcf-fbcc-41b1-bf9a-52b248656578"
+					(reference "J4")
+					(unit 1)
+				)

Commit message: 3dcad/housing: fdm & sla variants; kicad/power_supply: add p-down resistor to the MCP1640's EN pin
Parts:
- added R6: 309K, Resistor_SMD:R_0603_1608Metric, symbol Device:R
- R3: value 470R -> 200R
Connections:
- net GND: now also R6.2
- net at J4.1 (Pin_1), U1.3 (EN): now also R6.1
Changed lines of the file:
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@@
+	)
+	(junction
+		(at 101.6 146.05)
+		(diameter 0)
+		(color 0 0 0 0)
 	)
 	(junction
@@
 	)
 	(junction
+		(at 111.76 168.91)
+		(diameter 0)
+		(color 0 0 0 0)
+	)
+	(junction
 		(at 166.37 76.2)
 		(diameter 0)
@@
 	(wire
 		(pts
+			(xy 111.76 168.91) (xy 111.76 176.53)
+		)
+		(stroke
+			(width 0)
+			(type default)
+		)
+	)
+	(wire
+		(pts
 			(xy 139.7 151.13) (xy 165.1 151.13)
 		)
@@
 	(wire
 		(pts
-			(xy 111.76 151.13) (xy 111.76 153.67)
-		)
-		(stroke
-			(width 0)
-			(type default)
-		)
-	)
-	(wire
-		(pts
-			(xy 97.79 146.05) (xy 121.92 146.05)
+			(xy 111.76 151.13) (xy 111.76 168.91)
+		)
+		(stroke
+			(width 0)
+			(type default)
+		)
+	)
+	(wire
+		(pts
+			(xy 97.79 146.05) (xy 101.6 146.05)
 		)
 		(stroke
@@
 	(wire
 		(pts
+			(xy 101.6 146.05) (xy 101.6 153.67)
+		)
+		(stroke
+			(width 0)
+			(type default)
+		)
+	)
+	(wire
+		(pts
 			(xy 209.55 66.04) (xy 215.9 66.04)
 		)
@@
 	(wire
 		(pts
+			(xy 101.6 168.91) (xy 111.76 168.91)
+		)
+		(stroke
+			(width 0)
+			(type default)
+		)
+	)
+	(wire
+		(pts
 			(xy 234.95 69.85) (xy 234.95 76.2)
 		)
@@
 	(wire
 		(pts
+			(xy 101.6 161.29) (xy 101.6 168.91)
+		)
+		(stroke
+			(width 0)
+			(type default)
+		)
+	)
+	(wire
+		(pts
 			(xy 153.67 115.57) (xy 153.67 128.27)
 		)
@@
 		(pts
 			(xy 196.85 124.46) (xy 190.5 124.46)
+		)
+		(stroke
+			(width 0)
+			(type default)
+		)
+	)
+	(wire
+		(pts
+			(xy 101.6 146.05) (xy 121.92 146.05)
 		)
 		(stroke
@@
 	)
 	(symbol
+		(lib_id "Device:R")
+		(at 101.6 157.48 0)
+		(unit 1)
+		(exclude_from_sim no)
+		(in_bom yes)
+		(on_board yes)
+		(dnp no)
+		(fields_autoplaced yes)
+		(property "Reference" "R6"
+			(at 104.14 156.2099 0)
+			(effects
+				(font
+					(size 1.27 1.27)
+				)
+				(justify left)
+			)
+		)
+		(property "Value" "309K"
+			(at 104.14 158.7499 0)
+			(effects
+				(font
+					(size 1.27 1.27)
+				)
+				(justify left)
+			)
+		)
+		(property "Footprint" "Resistor_SMD:R_0603_1608Metric"
+			(at 99.822 157.48 90)
+			(effects
+				(font
+					(size 1.27 1.27)
+				)
+				(hide yes)
+			)
+		)
+		(property "Datasheet" "~"
+			(at 101.6 157.48 0)
+			(effects
+				(font
+					(size 1.27 1.27)
+				)
+				(hide yes)
+			)
+		)
+		(property "Description" "Resistor"
+			(at 101.6 157.48 0)
+			(effects
+				(font
+					(size 1.27 1.27)
+				)
+				(hide yes)
+			)
+		)
+		(pin "2"
+		)
+		(pin "1"
+		)
+		(instances
+			(project "power_supply"
+				(path "/5e0ffdcf-fbcc-41b1-bf9a-52b248656578"
+					(reference "R6")
+					(unit 1)
+				)
+			)
+		)
+	)
+	(symbol
 		(lib_id "Transistor_FET:DMG2301L")
 		(at 87.63 71.12 0)
@@
 			)
 		)
-		(property "Value" "470R"
+		(property "Value" "200R"
 			(at 205.74 62.23 90)
 			(effects
@@
 	(symbol
 		(lib_id "power:GND")
-		(at 111.76 153.67 0)
+		(at 111.76 176.53 0)
 		(unit 1)
 		(exclude_from_sim no)
@@
 		(dnp no)
 		(property "Reference" "#PWR01"
-			(at 111.76 160.02 0)
+			(at 111.76 182.88 0)
 			(effects
 				(font
@@
 		)
 		(property "Value" "GND"
-			(at 111.76 158.75 0)
+			(at 111.76 181.61 0)
 			(effects
 				(font
@@
 		)
 		(property "Footprint" ""
-			(at 111.76 153.67 0)
+			(at 111.76 176.53 0)
 			(effects
 				(font
@@
 		)
 		(property "Datasheet" ""
-			(at 111.76 153.67 0)
+			(at 111.76 176.53 0)
 			(effects
 				(font
@@
 		)
 		(property "Description" "Power symbol creates a global label with name \"GND\" , ground"
-			(at 111.76 153.67 0)
-			(effects
-				(font
+			(at 111.76 176.53 0)
+			(effects
+				(font
